Commit message: Everything Runs

File: src/vqwbot_bringup/urdf/vqwbot.inertia.xacro (robot description, xacro)
@@ -1,5 +1,4 @@
 <?xml version="1.0"?>
 <robot xmlns:xacro="http://www.ros.org/wiki/xacro">
-  <!-- Define inertial property macros  -->
   <xacro:macro name="box_inertia" params="m w h d">
     <inertial>

File: src/vqwbot_bringup/urdf/vqwbot.materials.xacro (robot description, xacro)
@@ -14,4 +14,10 @@
     <color rgba="0.0 0.8 0.0 1.0"/>
   </material>
+  <material name="yellow">
+    <color rgba="1.0 1.0 0.0 1.0"/>
+  </material>
+  <material name="yellow_transparent">
+    <color rgba="1.0 1.0 0.0 0.2"/>
+  </material>
   <material name="grey">
     <color rgba="0.2 0.2 0.2 1.0"/>
@@ -19,4 +25,7 @@
   <material name="orange">
     <color rgba="${255/255} ${108/255} ${10/255} 1.0"/>
+  </material>
+  <material name="orange_transparent">
+    <color rgba="${255/255} ${108/255} ${10/255} 0.2"/>
   </material>
   <material name="brown">

File: src/vqwbot_bringup/urdf/vqwbot.urdf.xacro (robot description, xacro)
@@ -1,8 +1,8 @@
 <?xml version="1.0"?>
-<!-- Basic differential drive mobile base -->
+<!-- vqwbot differential drive mobile base -->
 <robot xmlns:xacro="http://www.ros.org/wiki/xacro" name="vqwbot">
   <!-- Import Rviz colors -->
   <xacro:include filename="$(find vqwbot_bringup)/urdf/vqwbot.materials.xacro" />
-  <!-- Import inertia mscros -->
+  <!-- Import inertia macros -->
   <xacro:include filename="$(find vqwbot_bringup)/urdf/vqwbot.inertia.xacro" />
 <!-- import vqwbot_base macro -->
@@ -12,6 +12,13 @@
   <!-- Import bno08x_ros2_control macro -->
   <xacro:include filename="$(find vqwbot_bringup)/urdf/bno08x.ros2_control.xacro" />
+  <!-- Import camera_urdf macro -->
+  <xacro:include filename="$(find vqwbot_bringup)/urdf/camera.urdf.xacro" />
+  <!-- Import camera_urdf macro -->
+  <xacro:include filename="$(find vqwbot_bringup)/urdf/cam_pan_tilt_ros2_control.xacro" />
   <xacro:vqwbot_base />
+  <xacro:camera_urdf prefix="L" y_multiplier="1" />
+  <xacro:camera_urdf prefix="R" y_multiplier="-1" />
   <xacro:roboclaw_ros2_control name="roboclaw_controller" />
   <xacro:bno08x_ros2_control name="bno08x_controller" />
+  <!-- <xacro:cam_pan_tilt_ros2_control name="pan_tilt_controller" /> -->
 </robot>

File: src/vqwbot_bringup/urdf/vqwbot_description.urdf.xacro (robot description, xacro)
@@ -1,5 +1,4 @@
 <?xml version="1.0"?>
 <robot xmlns:xacro="http://www.ros.org/wiki/xacro">
-    <!-- <xacro:include filename="$(find vqwbot_bringup)/urdf/vqwbot.inertia.xacro" /> -->
   <xacro:macro name="vqwbot_base">
     <!-- Constants for robot dimensions -->
@@ -7,13 +6,14 @@
     <xacro:property name="base_mass" value="0.003" />
     <!-- TODO: Fixme -->
-    <xacro:property name="base_width" value="0.04" />
-    <xacro:property name="base_length" value="0.58" />
-    <xacro:property name="base_height" value="0.03" />
-    <xacro:property name="base1_width" value="0.33" />
-    <xacro:property name="base1_length" value="0.28" />
-    <xacro:property name="base1_height" value="0.08" />
+    <xacro:property name="base_width" value="0.32" />
+    <xacro:property name="base_length" value="0.24" />
+    <xacro:property name="base_height" value="0.07" />
     <xacro:property name="base2_width" value="0.30" />
     <xacro:property name="base2_length" value="0.25" />
     <xacro:property name="base2_height" value="0.12" />
+    <xacro:property name="tail_width" value="0.04" />
+    <xacro:property name="tail_length" value="0.25" />
+    <xacro:property name="tail_height" value="0.03" />
+    <xacro:property name="tail_offset" value="-0.13" />
     <xacro:property name="wheel_mass" value="0.001" />
     <xacro:property name="wheel_len" value="0.03" />
@@ -21,8 +21,11 @@
     <xacro:property name="caster_wheel_mass" value="0.0005" />  <!-- TODO: Fixme -->
     <xacro:property name="caster_wheel_radius" value="0.025" />
-    <xacro:property name="lidar_height" value="0.25" />
-    <xacro:property name="imu_height" value="0.12" />
-    <xacro:property name="wheel_from_centerline" value="${-base1_width/2 - wheel_len/2}" />
+    <xacro:property name="caster_wheel_x_offset" value="-0.200" />
+    <xacro:property name="lidar_height" value="0.39" />
+    <xacro:property name="imu_height" value="0.16" />
+    <xacro:property name="wheel_from_centerline" value="${-base_width/2 - wheel_len/2}" />
+    <!-- ======================================================================== -->
     <link name="base_footprint" />
+    <!-- ======================================================================== -->
     <joint name="base_joint" type="fixed">
       <parent link="base_footprint"/>
@@ -30,5 +33,5 @@
       <origin xyz="0 0 ${wheel_radius}" rpy="0 0 0"/>
     </joint>
-    <link name="base_link">
+    <link name="base_link"> <!-- this is the main body's box -->
       <collision>
         <origin xyz="0 0 ${(base_height/2)-(wheel_radius/2)}" rpy="0 0 0"/>
@@ -42,53 +45,56 @@
           <box size="${base_length} ${base_width} ${base_height}"/>
         </geometry>
-        <material name="orange"/>
-      </visual>
-      <xacro:box_inertia m="${base_mass}" w="${base_width}" h="${base_height}" d="${base_length}" />
-    </link>
-    <link name="base1_link">
-      <collision>
-        <origin xyz="0 0 ${(base1_height/2)-(wheel_radius/2)}" rpy="0 0 0"/>
-        <geometry>
-          <box size="${base1_length} ${base1_width} ${base1_height}"/>
-        </geometry>
-      </collision>
-      <visual>
-        <origin xyz="0 0 ${(base1_height/2)-(wheel_radius/2)}" rpy="0 0 0"/>
-        <geometry>
-          <box size="${base1_length} ${base1_width} ${base1_height}"/>
-        </geometry>
-        <material name="orange"/>
-      </visual>
-    </link>
-    <joint name="base1_joint" type="fixed">
-      <parent link="base_link"/>
-      <child link="base1_link"/>
+        <material name="yellow_transparent"/>
+      </visual>
+    </link>
+    <!-- ======================================================================== -->
+    <joint name="tail_joint" type="fixed">
+      <parent link="base_link"/>
+      <child link="tail_link"/>
       <origin xyz="0 0 0" rpy="0 0 0"/>
     </joint>
-    <link name="upper_base_link">
-      <collision>
-        <origin xyz="${(base2_width/2)} 0 ${(base1_height/2)+(base2_height/2)}" rpy="0 0 0"/>
-        <geometry>
-          <box size="${base2_length} ${base2_width} ${base2_height}"/>
-        </geometry>
-      </collision>
-      <visual>
-        <origin xyz="0 0 ${(base1_height/2)+(base2_height/2)}" rpy="0 0 0"/>
-        <geometry>
-          <box size="${base2_length} ${base2_width} ${base2_height}"/>
-        </geometry>
-        <material name="orange"/>
-      </visual>
-    </link>
+    <link name="tail_link"> <!-- this is Tail that sticks out of the back -->
+      <collision>
+        <origin xyz="${tail_offset} 0 ${(tail_height/2)-(wheel_radius/2)}" rpy="0 0 0"/>
+        <geometry>
+          <box size="${tail_length} ${tail_width} ${tail_height}"/>
+        </geometry>
+      </collision>
+      <visual>
+        <origin xyz="${tail_offset} 0 ${(tail_height/2)-(wheel_radius/2)}" rpy="0 0 0"/>
+        <geometry>
+          <box size="${tail_length} ${tail_width} ${tail_height}"/>
+        </geometry>
+        <material name="yellow_transparent"/>
+      </visual>
+      <xacro:box_inertia m="${base_mass}" w="${tail_width}" h="${tail_height}" d="${tail_length}" />
+    </link>
+    <!-- ======================================================================== -->
     <joint name="upper_base_joint" type="fixed">
-      <parent link="base1_link"/>
+      <parent link="base_link"/>
       <child link="upper_base_link"/>
       <origin xyz="0 0 0" rpy="0 0 0"/>
     </joint>
+    <link name="upper_base_link">
+      <collision>
+        <origin xyz="0 0 ${(base_height/2)+(base2_height/2)}" rpy="0 0 0"/>
+        <!-- <origin xyz="${(base2_width/2)} 0 ${(base_height/2)+(base2_height/2)}" rpy="0 0 0"/> -->
+        <geometry>
+          <box size="${base2_length} ${base2_width} ${base2_height}"/>
+        </geometry>
+      </collision>
+      <visual>
+        <origin xyz="0 0 ${(base_height/2)+(base2_height/2)}" rpy="0 0 0"/>
+        <geometry>
+          <box size="${base2_length} ${base2_width} ${base2_height}"/>
+        </geometry>
+        <material name="orange_transparent" />
+      </visual>
+    </link>
     <!-- ======================================================================== -->
     <joint name="left_wheel_joint" type="continuous">
       <parent link="base_link"/>
       <child link="left_wheel"/>
-      <origin xyz="0 ${-base1_width/2 - wheel_len/2} 0" rpy="0 0 0"/>
+      <origin xyz="0 ${-base_width/2 - wheel_len/2} 0" rpy="0 0 0"/>
       <axis xyz="0 1 0"/>
       <dynamics damping="0.2"/>
@@ -114,5 +120,5 @@
       <parent link="base_link"/>
       <child link="right_wheel"/>
-      <origin xyz="0 ${base1_width/2 + wheel_len/2} 0" rpy="0 0 0"/>
+      <origin xyz="0 ${base_width/2 + wheel_len/2} 0" rpy="0 0 0"/>
       <axis xyz="0 1 0"/>
       <dynamics damping="0.2"/>
@@ -138,5 +144,5 @@
       <parent link="base_link"/>
       <child link="caster_rear_wheel"/>
-      <origin xyz="${base_length/2} 0 ${caster_wheel_radius - wheel_radius}" rpy="0 0 0"/>
+      <origin xyz="${caster_wheel_x_offset} 0 ${caster_wheel_radius - wheel_radius}" rpy="0 0 0"/>
     </joint>
     <link name="caster_rear_wheel">
@@ -160,5 +166,5 @@
       <parent link="base_link"/>
       <child link="laser_scan"/>
-      <origin xyz="0 0 ${lidar_height}" rpy="0 0 0"/>
+      <origin xyz="0 0 ${lidar_height}" rpy="0 0 3.1415926"/>
     </joint>
     <link name="laser_scan">
@@ -172,5 +178,5 @@
         <origin xyz="0 0 0" rpy="0 0 0"/>
         <geometry>
-          <cylinder length="0.04" radius="0.05"/>
+          <cylinder length="0.03" radius="0.05"/>
         </geometry>
         <material name="red"/>
@@ -187,11 +193,11 @@
         <origin xyz="0 0 0" rpy="0 0 0"/>
         <geometry>
-          <cylinder length="0.04" radius="0.05"/>
-        </geometry>
-      </collision>
-      <visual>
-        <origin xyz="0 0 0" rpy="0 0 0"/>
-        <geometry>
-          <cylinder length="0.004" radius="0.005"/>
+          <cylinder length="0.004" radius="0.01"/>
+        </geometry>
+      </collision>
+      <visual>
+        <origin xyz="0 0 0" rpy="0 0 0"/>
+        <geometry>
+          <cylinder length="0.004" radius="0.01"/>
         </geometry>
         <material name="green"/>
