Commit message: will drive with joystick

File: src/vqwbot_bringup/urdf/cam_pan_tilt_ros2_control.xacro (robot description, xacro)
@@ -7,8 +7,8 @@
           <param name="i2c_device">/dev/i2c-1</param>
       </hardware>
-      <xacro:servo_ros2_control joint_name="camera_L_pan_joint" channel="0" />
-      <xacro:servo_ros2_control joint_name="camera_L_tilt_joint" channel="1" />
-      <xacro:servo_ros2_control joint_name="camera_R_pan_joint" channel="2" />
-      <xacro:servo_ros2_control joint_name="camera_R_tilt_joint" channel="3" />
+      <xacro:servo_ros2_control joint_name="camera_L_pan_joint" channel="12" offset="0.4" />
+      <xacro:servo_ros2_control joint_name="camera_L_tilt_joint" channel="13" offset="0.1" />
+      <xacro:servo_ros2_control joint_name="camera_R_pan_joint" channel="14" offset="-0.1" />
+      <xacro:servo_ros2_control joint_name="camera_R_tilt_joint" channel="15" offset="0.0" />
     </ros2_control>
   </xacro:macro>

File: src/vqwbot_bringup/urdf/servo_ros2_control.xacro (robot description, xacro)
@@ -1,7 +1,8 @@
 <?xml version="1.0"?>
 <robot xmlns:xacro="http://www.ros.org/wiki/xacro">
-  <xacro:macro name="servo_ros2_control" params="joint_name channel">
+  <xacro:macro name="servo_ros2_control" params="joint_name channel offset">
       <joint name="${joint_name}">
         <param name="channel">${channel}</param>
+        <param name="offset">${offset}</param>
         <command_interface name="position">
           <param name="min_position">-1.570796</param>

File: src/vqwbot_bringup/urdf/vqwbot.urdf.xacro (robot description, xacro)
@@ -14,5 +14,7 @@
   <!-- Import camera_urdf macro -->
   <xacro:include filename="$(find vqwbot_bringup)/urdf/camera.urdf.xacro" />
-  <!-- Import camera_urdf macro -->
+  <!-- Import servo_ros2_control macro -->
+  <xacro:include filename="$(find vqwbot_bringup)/urdf/servo_ros2_control.xacro" />
+  <!-- Import cam_pan_tilt_ros2_control macro -->
   <xacro:include filename="$(find vqwbot_bringup)/urdf/cam_pan_tilt_ros2_control.xacro" />
   <xacro:vqwbot_base />
@@ -21,4 +23,4 @@
   <xacro:roboclaw_ros2_control name="roboclaw_controller" />
   <xacro:bno08x_ros2_control name="bno08x_controller" />
-  <!-- <xacro:cam_pan_tilt_ros2_control name="pan_tilt_controller" /> -->
+  <xacro:cam_pan_tilt_ros2_control name="pan_tilt_controller" />
 </robot>

File: src/vqwbot_bringup/urdf/vqwbot_description.urdf.xacro (robot description, xacro)
@@ -26,5 +26,19 @@
     <xacro:property name="wheel_from_centerline" value="${-base_width/2 - wheel_len/2}" />
     <!-- ======================================================================== -->
-    <link name="base_footprint" />
+    <link name="base_footprint">
+      <collision>
+        <origin xyz="0 0 0" rpy="0 0 0"/>
+        <geometry>
+          <box size="${base_length} ${base_width} 0.001"/>
+        </geometry>
+      </collision>
+      <visual>
+        <origin xyz="0 0 0" rpy="0 0 0"/>
+        <geometry>
+          <box size="${base_length} ${base_width} 0.001"/>
+        </geometry>
+        <material name="orange_transparent"/>
+      </visual>
+    </link>
     <!-- ======================================================================== -->
     <joint name="base_joint" type="fixed">
@@ -96,5 +110,5 @@
       <parent link="base_link"/>
       <child link="left_wheel"/>
-      <origin xyz="0 ${-base_width/2 - wheel_len/2} 0" rpy="0 0 0"/>
+      <origin xyz="0 ${base_width/2 - wheel_len/2} 0" rpy="0 0 0"/>
       <axis xyz="0 1 0"/>
       <dynamics damping="0.2"/>
@@ -120,5 +134,5 @@
       <parent link="base_link"/>
       <child link="right_wheel"/>
-      <origin xyz="0 ${base_width/2 + wheel_len/2} 0" rpy="0 0 0"/>
+      <origin xyz="0 ${-base_width/2 + wheel_len/2} 0" rpy="0 0 0"/>
       <axis xyz="0 1 0"/>
       <dynamics damping="0.2"/>
