Commit message: launch stuff

File: src/vqwbot_bringup/urdf/vqwbot_description.urdf.xacro (robot description, xacro)
@@ -26,5 +26,5 @@
     <xacro:property name="wheel_from_centerline" value="${-base_width/2 - wheel_len/2}" />
     <!-- ======================================================================== -->
-    <link name="base_footprint">
+    <!-- <link name="base_footprint">
       <collision>
         <origin xyz="0 0 0" rpy="0 0 0"/>
@@ -40,11 +40,12 @@
         <material name="orange_transparent"/>
       </visual>
-    </link>
-    <!-- ======================================================================== -->
-    <joint name="base_joint" type="fixed">
+    </link> -->
+    <!-- ======================================================================== -->
+    <!-- ======================================================================== -->
+    <!-- <joint name="base_joint" type="fixed">
       <parent link="base_footprint"/>
       <child link="base_link"/>
       <origin xyz="0 0 ${wheel_radius}" rpy="0 0 0"/>
-    </joint>
+    </joint> -->
     <link name="base_link"> <!-- this is the main body's box -->
       <collision>
@@ -62,4 +63,26 @@
       </visual>
     </link>
+    <!-- ======================================================================== -->
+    <link name="base_footprint">
+      <collision>
+        <origin xyz="0 0 0" rpy="0 0 0"/>
+        <geometry>
+          <box size="${base_length} ${base_width} 0.001"/>
+        </geometry>
+      </collision>
+      <visual>
+        <origin xyz="0 0 0" rpy="0 0 0"/>
+        <geometry>
+          <box size="${base_length} ${base_width} 0.001"/>
+        </geometry>
+        <material name="orange_transparent"/>
+      </visual>
+    </link>
+    <!-- ======================================================================== -->
+    <joint name="base_footprint_joint" type="fixed">
+      <parent link="base_link"/>
+      <child link="base_footprint"/>
+      <origin xyz="0 0 0" rpy="0 0 0"/>
+    </joint>
     <!-- ======================================================================== -->
     <joint name="tail_joint" type="fixed">
